File: Hardware/Chameleon.sch (KiCad schematic (older format))
At the start: 24 parts

Commit message: Heavily updated schematics and Project Log
Parts:
- removed C? (x4): .1uF, symbol CSMALL
- removed U?: AS1107, symbol AS1107
- added C? (x3): CSMALL, symbol CSMALL
- added C? (x7): .1uF, symbol CSMALL
- added CS?: 10uF, symbol CSMALL
- added D?: LED, symbol LED
- added IC?: ATTINY44-SS, SO14, symbol ATTINY44-SS
- added L?: INDUCTOR, symbol INDUCTOR
- added P?: CONN_3X2, symbol CONN_3X2
- added R? (x5): 10k, symbol R
- added R? (x6): 220, symbol R
- added R? (x10): 150, symbol R
- added U?: PCA9635, symbol PCA9635
- added X?: CRYSTAL, symbol CRYSTAL
- BT?: value BATTERY -> 4.2V 500mAh
- CS0: renamed from C?; value CS0 -> 4.7nF
Connections:
- net labels added: MISO, MOSI, RESET, SCK, VCC, XTAL1, XTAL2
- wire segments 85 -> 220
Other:
- note added: "Crystal and Load Caps"
- moved on the sheet: BT?, LED?, RX0, RY0, RYB0, S?

Commit message: Made several updates to BOM, Project Log, and Schematics
Parts:
- removed U?: SPX29150T-L-5-0/TR, symbol SPX29150T-L-5-0/TR
- BT?: value 4.2V 500mAh -> 3.7V 500mAh
- L?: value INDUCTOR -> 33uH
Changed lines of the file:
@@
-EESchema Schematic File Version 2  date 5/7/2012 4:34:33 PM
+EESchema Schematic File Version 2  date 5/12/2012 11:31:01 AM
 LIBS:power
 LIBS:device
@@
 Sheet 1 1
 Title "Chameleon drink coasters"
-Date "7 may 2012"
+Date "12 may 2012"
 Rev "1.0"
 Comp "Projects and Stuff LLC"
@@
 P 750 1050
 F 0 "L?" V 700 1050 40  0000 C CNN
-F 1 "INDUCTOR" V 850 1050 40  0000 C CNN
+F 1 "33uH" V 850 1050 40  0000 C CNN
 	1    750  1050
 	1    0    0    -1
@@
 6E 56 52 49 51 4E 59 71 7E 65 C5 4D 0F AF 00 BF F6 21 9D BA 45 88 9C 00 16 00 C0 66 90 E0 00 00
 AC 42 3B 38 00 00 AB 90 E0 00 00 AC 42 82 03 00 B0 EA FF 00 E3 76 B5 A7 81 B6 BC 08 00 00 00 00
-49 45 4E 44 AE 42 60 82 11 $EndBitmap
+49 45 4E 44 AE 42 60 82 83 $EndBitmap
 EndData
 $EndBitmap
@@
 P 8300 1350
 F 0 "BT?" H 8300 1550 50  0000 C CNN
-F 1 "4.2V 500mAh" H 8300 1160 50  0000 C CNN
+F 1 "3.7V 500mAh" H 8300 1160 50  0000 C CNN
 	1    8300 1350
 	0    -1   -1   0
 $EndComp
-$Comp
-L SPX29150T-L-5-0/TR U?
-U 1 1 4FA6C810
-P 9700 1000
-F 0 "U?" H 10000 600 60  0000 C CNN
-F 1 "SPX29150T-L-5-0/TR" H 9700 1150 60  0000 C CNN
-	1    9700 1000
-	1    0    0    -1
-$EndComp
 $EndSCHEMATC

Commit message: Updated Schematics with Boost regulator and PCA9685
Parts:
- removed C? (x3): .1uF, symbol CSMALL
- removed U?: PCA9635, symbol PCA9635
- added D?: DIODESCH, symbol DIODESCH
- added L?: 47uH, symbol INDUCTOR
- added U?: NCP1402, symbol NCP1402
- added U?: PCA9685, symbol PCA9685
- C?: value 10uF -> 47uF
Connections:
- net labels removed: +5V
- wire segments 220 -> 223
- no-connect marks 0 -> 1
Other:
- note added: "Input Power & Regulation Block"
- moved on the sheet: BT?, RX0, RY0, RYB0, X?

Commit message: Updated Schematics with USB connector, and updated BOM and Project Log
Parts:
- added S?: TL3315NF160Q, symbol TL3315NF160Q
- added U?: USBMICRO-B, symbol USBMICRO-B
- C?: value CSMALL -> .1uF
- C? (x2): value CSMALL -> 8pF
Connections:
- wire segments 223 -> 236
- no-connect marks 1 -> 4
Other:
- moved on the sheet: BT?, D?, L?, U?
Changed lines of the file:
@@
-EESchema Schematic File Version 2  date 5/12/2012 3:14:52 PM
+EESchema Schematic File Version 2  date 5/12/2012 6:42:25 PM
 LIBS:power
 LIBS:device
@@
 Comment4 ""
 $EndDescr
-Text Notes 7250 900  0    60   ~ 0
-Input Power & Regulation Block
-Wire Bus Line
-	7250 3000 10200 3000
-Wire Bus Line
-	10200 3000 10200 900
-Wire Bus Line
-	10200 900  7250 900
+Connection ~ 3500 2100
+Connection ~ 3450 2700
+Wire Wire Line
+	3450 2700 3450 2500
+Wire Wire Line
+	3500 2500 3450 2500
+Wire Wire Line
+	3500 2050 3500 2500
+Connection ~ 3450 3500
+Wire Wire Line
+	3450 3550 3450 3500
+Wire Notes Line
+	4850 3000 11100 3000
+Wire Wire Line
+	8300 2500 9500 2500
+Wire Wire Line
+	8300 2500 8300 2300
+Wire Wire Line
+	8300 2300 8100 2300
 Wire Bus Line
 	7250 900  7250 1950
@@
 Wire Wire Line
 	2400 6650 2400 6100
-Connection ~ 8600 1850
-Wire Wire Line
-	8600 1850 8600 1550
-Wire Wire Line
-	8600 1550 8950 1550
-Wire Wire Line
-	9650 2050 9700 2050
-Wire Wire Line
-	7600 2600 7600 2500
-Connection ~ 7900 1850
-Wire Wire Line
-	7900 1900 7900 1850
-Wire Wire Line
-	2900 2100 3500 2100
-Wire Wire Line
-	3500 2100 3500 2050
+Connection ~ 9550 1800
+Wire Wire Line
+	9550 1800 9550 1500
+Wire Wire Line
+	9550 1500 9900 1500
+Wire Wire Line
+	10600 2000 10650 2000
+Wire Wire Line
+	8550 2550 8550 2450
+Connection ~ 8850 1800
+Wire Wire Line
+	8850 1850 8850 1800
+Wire Wire Line
+	3500 2100 2900 2100
 Wire Wire Line
 	2900 1600 2950 1600
@@
 	6950 4050 6950 4100
 Wire Wire Line
-	9850 2100 9850 2150
-Wire Wire Line
-	7900 2100 7900 2150
+	10800 2050 10800 2100
+Wire Wire Line
+	8850 2050 8850 2100
 Wire Wire Line
 	5650 1200 5750 1200
@@
 Wire Notes Line
 	7250 1950 7250 3000
-Wire Notes Line
-	7250 3000 4850 3000
 Wire Wire Line
 	3950 2650 3950 2700
@@
 	3500 1550 3500 1500
 Wire Wire Line
-	7600 1900 7600 1850
-Wire Wire Line
-	7600 1850 7950 1850
-Wire Wire Line
-	8550 1850 8650 1850
-Wire Wire Line
-	8650 2050 8550 2050
-Wire Wire Line
-	8550 2050 8550 2550
-Wire Wire Line
-	8550 2550 7600 2550
-Connection ~ 7600 2550
-Wire Wire Line
-	9350 1550 9700 1550
-Wire Wire Line
-	9700 1550 9700 2050
-Connection ~ 9700 1850
-Wire Wire Line
-	9650 1850 9850 1850
-Wire Wire Line
-	9850 1850 9850 1900
+	8550 1800 8550 1850
+Wire Wire Line
+	9500 1800 9600 1800
+Wire Wire Line
+	9600 2000 9500 2000
+Wire Wire Line
+	9500 2000 9500 2500
+Connection ~ 8550 2500
+Wire Wire Line
+	10300 1500 10650 1500
+Wire Wire Line
+	10650 1500 10650 2000
+Connection ~ 10650 1800
+Wire Wire Line
+	10600 1800 10800 1800
+Wire Wire Line
+	10800 1800 10800 1850
 Wire Wire Line
 	2300 5050 2300 4900
@@
 Connection ~ 2100 4900
 Connection ~ 2300 5000
+Wire Wire Line
+	8100 1900 8300 1900
+Wire Wire Line
+	8300 1900 8300 1800
+Wire Wire Line
+	8300 1800 8900 1800
+Connection ~ 8550 1800
+Wire Notes Line
+	7250 900  11100 900
+Wire Notes Line
+	11100 900  11100 3000
+Wire Wire Line
+	3350 3450 3350 3500
+Wire Wire Line
+	3350 3500 3550 3500
+Wire Wire Line
+	3550 3500 3550 3450
+Wire Wire Line
+	3350 2750 3350 2700
+Wire Wire Line
+	3350 2700 3550 2700
+Wire Wire Line
+	3550 2700 3550 2750
+$Comp
+L GND #PWR?
+U 1 1 4FAEE6FD
+P 3450 3550
+F 0 "#PWR?" H 3450 3550 30  0001 C CNN
+F 1 "GND" H 3450 3480 30  0001 C CNN
+	1    3450 3550
+	1    0    0    -1
+$EndComp
+$Comp
+L TL3315NF160Q S?
+U 1 1 4FAEE6F0
+P 3450 3100
+F 0 "S?" H 3500 2950 60  0000 C CNN
+F 1 "TL3315NF160Q" H 3350 3300 60  0000 C CNN
+	1    3450 3100
+	0    -1   -1   0
+$EndComp
+NoConn ~ 8100 2200
+NoConn ~ 8100 2100
+NoConn ~ 8100 2000
+$Comp
+L USBMICRO-B U?
+U 1 1 4FAEE647
+P 7800 2100
+F 0 "U?" H 7700 1800 60  0000 C CNN
+F 1 "USBMICRO-B" H 7650 2400 60  0000 C CNN
+	1    7800 2100
+	1    0    0    -1
+$EndComp
+Text Notes 7250 900  0    60   ~ 0
+Input Power & Regulation Block
 Text Label 2500 5950 0    60   ~ 0
 VCC
@@
 	1    0    0    -1
 $EndComp
-NoConn ~ 8650 1950
+NoConn ~ 9600 1900
 Text Label 1900 4850 0    60   ~ 0
 VCC
@@
 Text Label 750  700  0    60   ~ 0
 VCC
-Text Label 9850 1850 0    60   ~ 0
+Text Label 10800 1800 0    60   ~ 0
 VCC
 $Comp
 L DIODESCH D?
 U 1 1 4FAEB189
-P 9150 1550
-F 0 "D?" H 9150 1650 40  0000 C CNN
-F 1 "DIODESCH" H 9150 1450 40  0000 C CNN
-	1    9150 1550
+P 10100 1500
+F 0 "D?" H 10100 1600 40  0000 C CNN
+F 1 "DIODESCH" H 10100 1400 40  0000 C CNN
+	1    10100 1500
 	1    0    0    -1
 $EndComp
@@
 L INDUCTOR L?
 U 1 1 4FAEB118
-P 8250 1850
-F 0 "L?" V 8200 1850 40  0000 C CNN
-F 1 "47uH" V 8350 1850 40  0000 C CNN
-	1    8250 1850
+P 9200 1800
+F 0 "L?" V 9150 1800 40  0000 C CNN
+F 1 "47uH" V 9300 1800 40  0000 C CNN
+	1    9200 1800
 	0    -1   -1   0
 $EndComp
@@
 L NCP1402 U?
 U 1 1 4FAEB0F4
-P 9150 1950
-F 0 "U?" H 9250 1750 60  0000 C CNN
-F 1 "NCP1402" H 9150 2150 60  0000 C CNN
-	1    9150 1950
+P 10100 1900
+F 0 "U?" H 10200 1700 60  0000 C CNN
+F 1 "NCP1402" H 10100 2100 60  0000 C CNN
+	1    10100 1900
 	1    0    0    -1
 $EndComp
@@
 L GND #PWR?
 U 1 1 4FA82F70
-P 7600 2600
-F 0 "#PWR?" H 7600 2600 30  0001 C CNN
-F 1 "GND" H 7600 2530 30  0001 C CNN
-	1    7600 2600
+P 8550 2550
+F 0 "#PWR?" H 8550 2550 30  0001 C CNN
+F 1 "GND" H 8550 2480 30  0001 C CNN
+	1    8550 2550
 	1    0    0    -1
 $EndComp
@@
 P 6850 2900
 F 0 "C?" H 6875 2950 30  0000 L CNN
-F 1 "CSMALL" H 6875 2850 30  0000 L CNN
+F 1 "8pF" H 6875 2850 30  0000 L CNN
 	1    6850 2900
 	0    -1   -1   0
@@
 P 6850 2200
 F 0 "C?" H 6875 2250 30  0000 L CNN
-F 1 "CSMALL" H 6875 2150 30  0000 L CNN
+F 1 "8pF" H 6875 2150 30  0000 L CNN
 	1    6850 2200
 	0    -1   -1   0
@@
 P 750 1550
 F 0 "C?" H 775 1600 30  0000 L CNN
-F 1 "CSMALL" H 775 1500 30  0000 L CNN
+F 1 ".1uF" H 775 1500 30  0000 L CNN
 	1    750  1550
 	1    0    0    -1
@@
 6E 56 52 49 51 4E 59 71 7E 65 C5 4D 0F AF 00 BF F6 21 9D BA 45 88 9C 00 16 00 C0 66 90 E0 00 00
 AC 42 3B 38 00 00 AB 90 E0 00 00 AC 42 82 03 00 B0 EA FF 00 E3 76 B5 A7 81 B6 BC 08 00 00 00 00
-49 45 4E 44 AE 42 60 82 8F $EndBitmap
+49 45 4E 44 AE 42 60 82 D8 $EndBitmap
 EndData
 $EndBitmap
@@
 L GND #PWR?
 U 1 1 4FA6C9BD
-P 7900 2150
-F 0 "#PWR?" H 7900 2150 30  0001 C CNN
-F 1 "GND" H 7900 2080 30  0001 C CNN
-	1    7900 2150
+P 8850 2100
+F 0 "#PWR?" H 8850 2100 30  0001 C CNN
+F 1 "GND" H 8850 2030 30  0001 C CNN
+	1    8850 2100
 	1    0    0    -1
 $EndComp
@@
 L GND #PWR?
 U 1 1 4FA6C9B8
-P 9850 2150
-F 0 "#PWR?" H 9850 2150 30  0001 C CNN
-F 1 "GND" H 9850 2080 30  0001 C CNN
-	1    9850 2150
+P 10800 2100
+F 0 "#PWR?" H 10800 2100 30  0001 C CNN
+F 1 "GND" H 10800 2030 30  0001 C CNN
+	1    10800 2100
 	1    0    0    -1
 $EndComp
@@
 L CSMALL C?
 U 1 1 4FA6C832
-P 9850 2000
-F 0 "C?" H 9875 2050 30  0000 L CNN
-F 1 "47uF" H 9875 1950 30  0000 L CNN
-	1    9850 2000
+P 10800 1950
+F 0 "C?" H 10825 2000 30  0000 L CNN
+F 1 "47uF" H 10825 1900 30  0000 L CNN
+	1    10800 1950
 	1    0    0    -1
 $EndComp
@@
 L CSMALL C?
 U 1 1 4FA6C82E
-P 7900 2000
-F 0 "C?" H 7925 2050 30  0000 L CNN
-F 1 "10uF" H 7925 1950 30  0000 L CNN
-	1    7900 2000
+P 8850 1950
+F 0 "C?" H 8875 2000 30  0000 L CNN
+F 1 "10uF" H 8875 1900 30  0000 L CNN
+	1    8850 1950
 	1    0    0    -1
 $EndComp
@@
 L BATTERY BT?
 U 1 1 4FA6C819
-P 7600 2200
-F 0 "BT?" H 7600 2400 50  0000 C CNN
-F 1 "3.7V 500mAh" H 7600 2010 50  0000 C CNN
-	1    7600 2200
-	0    -1   -1   0
-$EndComp
+P 8550 2150
+F 0 "BT?" H 8550 2350 50  0000 C CNN
+F 1 "3.7V 500mAh" H 8550 1960 50  0000 C CNN
+	1    8550 2150
+	0    -1   -1   0
+$EndComp

Commit message: Annotated Schematics and finalized BOM
Parts:
- added TP1, TP2, TP3: TST, symbol TST
- L2: renamed from L?; value 47uH -> 33uH
- gave numbers to parts that had none: 52
- renumbered XOYO to XOYO1
Connections:
- net labels added: AIN0, MODE
- wire segments 236 -> 238
Other:
- note added: "ISP Header"
- moved on the sheet: IC1, L1, P1, R4, R5, RX0, RY0, RYB0, S1, S2, X1

Commit message: Wow, almost 4am. Worked on PCB layout. Needs more work. Components too close together
Parts:
- removed TP3: TST, symbol TST
Connections:
- wire segments 238 -> 237
Changed lines of the file:
@@
-EESchema Schematic File Version 2  date 5/12/2012 9:01:35 PM
+EESchema Schematic File Version 2  date 5/13/2012 2:38:40 AM
 LIBS:power
 LIBS:device
@@
 Wire Wire Line
 	8550 1750 8550 1850
-Wire Wire Line
-	9300 3700 9300 3750
-Connection ~ 9300 3750
 Wire Notes Line
 	11100 900  4450 900
@@
 Text Notes 5750 1000 0    60   ~ 0
 ISP Header
-$Comp
-L TST TP3
-U 1 1 4FAEFE3F
-P 9300 3700
-F 0 "TP3" H 9300 4000 40  0000 C CNN
-F 1 "TST" H 9300 3950 30  0000 C CNN
-	1    9300 3700
-	1    0    0    -1
-$EndComp
 $Comp
 L TST TP1
@@
 6E 56 52 49 51 4E 59 71 7E 65 C5 4D 0F AF 00 BF F6 21 9D BA 45 88 9C 00 16 00 C0 66 90 E0 00 00
 AC 42 3B 38 00 00 AB 90 E0 00 00 AC 42 82 03 00 B0 EA FF 00 E3 76 B5 A7 81 B6 BC 08 00 00 00 00
-49 45 4E 44 AE 42 60 82 B1 $EndBitmap
+49 45 4E 44 AE 42 60 82 C3 $EndBitmap
 EndData
 $EndBitmap

Commit message: Corrected the majority of known issues in Schematics and PCB, and updated BOM and Project Log
Parts:
- removed D1: DIODESCH, symbol DIODESCH
- removed R3: 10k, symbol R
- added D1: DIODESCH_MOD, symbol DIODESCH_MOD
- R1, R2: value 10k -> 1.5k
- R10, R6, R7, R8, R9: value 220 -> 320
- R11: value 220 -> 330
- R12, R13, R14, R15, R16, R17, R18, R19, R20, R21: value 150 -> 220
Connections:
- wire segments 237 -> 236
Changed lines of the file:
@@
-EESchema Schematic File Version 2  date 5/13/2012 2:38:40 AM
+EESchema Schematic File Version 2  date 8/13/2012 5:06:37 PM
 LIBS:power
 LIBS:device
@@
 Sheet 1 1
 Title "Chameleon Drink Coasters"
-Date "13 may 2012"
+Date "13 aug 2012"
 Rev "1.0"
 Comp "Projects and Stuff LLC"
@@
 $EndDescr
 Wire Wire Line
+	2100 5750 2100 5500
+Wire Wire Line
 	8850 1850 8850 1800
 Wire Notes Line
@@
 	1700 5700 2550 5700
 Wire Wire Line
-	2550 5500 2100 5500
-Wire Wire Line
-	2100 5500 2100 5450
+	2100 5500 2550 5500
 Wire Wire Line
 	8650 3550 8650 3600
@@
 	1700 4950 1700 4900
 Wire Wire Line
-	2100 4900 2100 4950
-Wire Wire Line
 	1900 4850 1900 4950
 Wire Wire Line
@@
 Wire Wire Line
 	2300 4900 1700 4900
-Connection ~ 2100 4900
 Connection ~ 2300 5000
 Wire Wire Line
@@
 Wire Wire Line
 	8300 1800 8900 1800
+$Comp
+L GND #PWR01
+U 1 1 5029561A
+P 2100 5750
+F 0 "#PWR01" H 2100 5750 30  0001 C CNN
+F 1 "GND" H 2100 5680 30  0001 C CNN
+	1    2100 5750
+	1    0    0    -1
+$EndComp
+$Comp
+L DIODESCH_MOD D1
+U 1 1 50294AD3
+P 10100 1500
+F 0 "D1" H 10100 1375 60  0000 C CNN
+F 1 "DIODESCH_MOD" H 10100 1625 60  0000 C CNN
+	1    10100 1500
+	1    0    0    -1
+$EndComp
 Text Label 2900 2100 0    60   ~ 0
 MODE
@@
 $EndComp
 $Comp
-L GND #PWR5
+L GND #PWR02
 U 1 1 4FAEE6FD
 P 3400 3550
-F 0 "#PWR5" H 3400 3550 30  0001 C CNN
+F 0 "#PWR02" H 3400 3550 30  0001 C CNN
 F 1 "GND" H 3400 3480 30  0001 C CNN
 	1    3400 3550
@@
 VCC
 $Comp
-L DIODESCH D1
-U 1 1 4FAEB189
-P 10100 1500
-F 0 "D1" H 10100 1600 40  0000 C CNN
-F 1 "DIODESCH" H 10100 1400 40  0000 C CNN
-	1    10100 1500
-	1    0    0    -1
-$EndComp
-$Comp
 L INDUCTOR L2
 U 1 1 4FAEB118
@@
 Y0B
 $Comp
-L GND #PWR10
+L GND #PWR03
 U 1 1 4FA82F70
 P 8550 2550
-F 0 "#PWR10" H 8550 2550 30  0001 C CNN
+F 0 "#PWR03" H 8550 2550 30  0001 C CNN
 F 1 "GND" H 8550 2480 30  0001 C CNN
 	1    8550 2550
@@
 P 1700 5200
 F 0 "R1" V 1780 5200 50  0000 C CNN
-F 1 "10k" V 1700 5200 50  0000 C CNN
+F 1 "1.5k" V 1700 5200 50  0000 C CNN
 	1    1700 5200
 	-1   0    0    1
@@
 P 1900 5200
 F 0 "R2" V 1980 5200 50  0000 C CNN
-F 1 "10k" V 1900 5200 50  0000 C CNN
+F 1 "1.5k" V 1900 5200 50  0000 C CNN
 	1    1900 5200
 	-1   0    0    1
 $EndComp
-Text Label 2500 5500 2    60   ~ 0
-RESET
-$Comp
-L R R3
-U 1 1 4FA82E27
-P 2100 5200
-F 0 "R3" V 2180 5200 50  0000 C CNN
-F 1 "10k" V 2100 5200 50  0000 C CNN
-	1    2100 5200
-	-1   0    0    1
-$EndComp
-$Comp
-L GND #PWR11
+$Comp
+L GND #PWR04
 U 1 1 4FA82A89
 P 8650 3600
-F 0 "#PWR11" H 8650 3600 30  0001 C CNN
+F 0 "#PWR04" H 8650 3600 30  0001 C CNN
 F 1 "GND" H 8650 3530 30  0001 C CNN
 	1    8650 3600
@@
 XTAL1
 $Comp
-L GND #PWR7
+L GND #PWR05
 U 1 1 4FA825F5
 P 6850 2550
-F 0 "#PWR7" H 6850 2550 30  0001 C CNN
+F 0 "#PWR05" H 6850 2550 30  0001 C CNN
 F 1 "GND" H 6850 2480 30  0001 C CNN
 	1    6850 2550
@@
 GND
 $Comp
-L GND #PWR2
+L GND #PWR06
 U 1 1 4FA82468
 P 2300 5350
-F 0 "#PWR2" H 2300 5350 30  0001 C CNN
+F 0 "#PWR06" H 2300 5350 30  0001 C CNN
 F 1 "GND" H 2300 5280 30  0001 C CNN
 	1    2300 5350
@@
 $EndComp
 $Comp
-L GND #PWR3
+L GND #PWR07
 U 1 1 4FA82417
 P 2400 6650
-F 0 "#PWR3" H 2400 6650 30  0001 C CNN
+F 0 "#PWR07" H 2400 6650 30  0001 C CNN
 F 1 "GND" H 2400 6580 30  0001 C CNN
 	1    2400 6650
@@
 P 5750 7000
 F 0 "R11" V 5830 7000 50  0000 C CNN
-F 1 "220" V 5750 7000 50  0000 C CNN
+F 1 "330" V 5750 7000 50  0000 C CNN
 	1    5750 7000
 	0    -1   -1   0
 $EndComp
 $Comp
-L GND #PWR17
+L GND #PWR08
 U 1 1 4FA81D5A
 P 10950 4100
-F 0 "#PWR17" H 10950 4100 30  0001 C CNN
+F 0 "#PWR08" H 10950 4100 30  0001 C CNN
 F 1 "GND" H 10950 4030 30  0001 C CNN
 	1    10950 4100
@@
 P 5750 6700
 F 0 "R10" V 5830 6700 50  0000 C CNN
-F 1 "220" V 5750 6700 50  0000 C CNN
+F 1 "320" V 5750 6700 50  0000 C CNN
 	1    5750 6700
 	0    -1   -1   0
@@
 P 6200 6800
 F 0 "R16" V 6280 6800 50  0000 C CNN
-F 1 "150" V 6200 6800 50  0000 C CNN
+F 1 "220" V 6200 6800 50  0000 C CNN
 	1    6200 6800
 	0    -1   -1   0
@@
 P 6650 6900
 F 0 "R21" V 6730 6900 50  0000 C CNN
-F 1 "150" V 6650 6900 50  0000 C CNN
+F 1 "220" V 6650 6900 50  0000 C CNN
 	1    6650 6900
 	0    -1   -1   0
@@
 P 5750 5500
 F 0 "R6" V 5830 5500 50  0000 C CNN
-F 1 "220" V 5750 5500 50  0000 C CNN
+F 1 "320" V 5750 5500 50  0000 C CNN
 	1    5750 5500
 	0    -1   -1   0
@@
 P 6200 5600
 F 0 "R12" V 6280 5600 50  0000 C CNN
-F 1 "150" V 6200 5600 50  0000 C CNN
+F 1 "220" V 6200 5600 50  0000 C CNN
 	1    6200 5600
 	0    -1   -1   0
@@
 P 6650 5700
 F 0 "R17" V 6730 5700 50  0000 C CNN
-F 1 "150" V 6650 5700 50  0000 C CNN
+F 1 "220" V 6650 5700 50  0000 C CNN
 	1    6650 5700
 	0    -1   -1   0
@@
 P 5750 5800
 F 0 "R7" V 5830 5800 50  0000 C CNN
-F 1 "220" V 5750 5800 50  0000 C CNN
+F 1 "320" V 5750 5800 50  0000 C CNN
 	1    5750 5800
 	0    -1   -1   0
@@
 P 6200 5900
 F 0 "R13" V 6280 5900 50  0000 C CNN
-F 1 "150" V 6200 5900 50  0000 C CNN
+F 1 "220" V 6200 5900 50  0000 C CNN
 	1    6200 5900
 	0    -1   -1   0
@@
 P 6650 6000
 F 0 "R18" V 6730 6000 50  0000 C CNN
-F 1 "150" V 6650 6000 50  0000 C CNN
+F 1 "220" V 6650 6000 50  0000 C CNN
 	1    6650 6000
 	0    -1   -1   0
@@
 P 6650 6600
 F 0 "R20" V 6730 6600 50  0000 C CNN
-F 1 "150" V 6650 6600 50  0000 C CNN
+F 1 "220" V 6650 6600 50  0000 C CNN
 	1    6650 6600
 	0    -1   -1   0
@@
 P 6200 6500
 F 0 "R15" V 6280 6500 50  0000 C CNN
-F 1 "150" V 6200 6500 50  0000 C CNN
+F 1 "220" V 6200 6500 50  0000 C CNN
 	1    6200 6500
 	0    -1   -1   0
@@
 P 5750 6400
 F 0 "R9" V 5830 6400 50  0000 C CNN
-F 1 "220" V 5750 6400 50  0000 C CNN
+F 1 "320" V 5750 6400 50  0000 C CNN
 	1    5750 6400
 	0    -1   -1   0
@@
 P 6650 6300
 F 0 "R19" V 6730 6300 50  0000 C CNN
-F 1 "150" V 6650 6300 50  0000 C CNN
+F 1 "220" V 6650 6300 50  0000 C CNN
 	1    6650 6300
 	0    -1   -1   0
@@
 P 6200 6200
 F 0 "R14" V 6280 6200 50  0000 C CNN
-F 1 "150" V 6200 6200 50  0000 C CNN
+F 1 "220" V 6200 6200 50  0000 C CNN
 	1    6200 6200
 	0    -1   -1   0
@@
 P 5750 6100
 F 0 "R8" V 5830 6100 50  0000 C CNN
-F 1 "220" V 5750 6100 50  0000 C CNN
+F 1 "320" V 5750 6100 50  0000 C CNN
 	1    5750 6100
 	0    -1   -1   0
@@
 $EndComp
 $Comp
-L GND #PWR15
+L GND #PWR09
 U 1 1 4FA8183F
 P 10350 4100
-F 0 "#PWR15" H 10350 4100 30  0001 C CNN
+F 0 "#PWR09" H 10350 4100 30  0001 C CNN
 F 1 "GND" H 10350 4030 30  0001 C CNN
 	1    10350 4100
@@
 $EndComp
 $Comp
-L GND #PWR12
+L GND #PWR010
 U 1 1 4FA8183B
 P 8650 4100
-F 0 "#PWR12" H 8650 4100 30  0001 C CNN
+F 0 "#PWR010" H 8650 4100 30  0001 C CNN
 F 1 "GND" H 8650 4030 30  0001 C CNN
 	1    8650 4100
@@
 $EndComp
 $Comp
-L GND #PWR14
+L GND #PWR011
 U 1 1 4FA8183A
 P 9500 4100
-F 0 "#PWR14" H 9500 4100 30  0001 C CNN
+F 0 "#PWR011" H 9500 4100 30  0001 C CNN
 F 1 "GND" H 9500 4030 30  0001 C CNN
 	1    9500 4100
@@
 $EndComp
 $Comp
-L GND #PWR9
+L GND #PWR012
 U 1 1 4FA81830
 P 7800 4100
-F 0 "#PWR9" H 7800 4100 30  0001 C CNN
+F 0 "#PWR012" H 7800 4100 30  0001 C CNN
 F 1 "GND" H 7800 4030 30  0001 C CNN
 	1    7800 4100
@@
 $EndComp
 $Comp
-L GND #PWR1
+L GND #PWR013
 U 1 1 4FA81791
 P 700 2650
-F 0 "#PWR1" H 700 2650 30  0001 C CNN
+F 0 "#PWR013" H 700 2650 30  0001 C CNN
 F 1 "GND" H 700 2580 30  0001 C CNN
 	1    700  2650
@@
 $EndComp
 $Comp
-L GND #PWR4
+L GND #PWR014
 U 1 1 4FA81695
 P 3300 1550
-F 0 "#PWR4" H 3300 1550 30  0001 C CNN
+F 0 "#PWR014" H 3300 1550 30  0001 C CNN
 F 1 "GND" H 3300 1480 30  0001 C CNN
 	1    3300 1550
@@
 $EndComp
 $Comp
-L GND #PWR6
+L GND #PWR015
 U 1 1 4FA8165E
 P 4050 3550
-F 0 "#PWR6" H 4050 3550 30  0001 C CNN
+F 0 "#PWR015" H 4050 3550 30  0001 C CNN
 F 1 "GND" H 4050 3480 30  0001 C CNN
 	1    4050 3550
@@
 6E 56 52 49 51 4E 59 71 7E 65 C5 4D 0F AF 00 BF F6 21 9D BA 45 88 9C 00 16 00 C0 66 90 E0 00 00
 AC 42 3B 38 00 00 AB 90 E0 00 00 AC 42 82 03 00 B0 EA FF 00 E3 76 B5 A7 81 B6 BC 08 00 00 00 00
-49 45 4E 44 AE 42 60 82 C3 $EndBitmap
+49 45 4E 44 AE 42 60 82 E8 $EndBitmap
 EndData
 $EndBitmap
@@
 $EndComp
 $Comp
-L GND #PWR8
+L GND #PWR016
 U 1 1 4FA6CB58
 P 6950 4100
-F 0 "#PWR8" H 6950 4100 30  0001 C CNN
+F 0 "#PWR016" H 6950 4100 30  0001 C CNN
 F 1 "GND" H 6950 4030 30  0001 C CNN
 	1    6950 4100
@@
 $EndComp
 $Comp
-L GND #PWR13
+L GND #PWR017
 U 1 1 4FA6C9BD
 P 8850 2100
-F 0 "#PWR13" H 8850 2100 30  0001 C CNN
+F 0 "#PWR017" H 8850 2100 30  0001 C CNN
 F 1 "GND" H 8850 2030 30  0001 C CNN
 	1    8850 2100
@@
 $EndComp
 $Comp
-L GND #PWR16
+L GND #PWR018
 U 1 1 4FA6C9B8
 P 10800 2100
-F 0 "#PWR16" H 10800 2100 30  0001 C CNN
+F 0 "#PWR018" H 10800 2100 30  0001 C CNN
 F 1 "GND" H 10800 2030 30  0001 C CNN
 	1    10800 2100
