File: Hardware/Chameleon.sch (KiCad schematic (older format))
At the start: 43 parts, among them P1 PDI, U2 USBMICRO-B, U3 NCP1402

Commit message: Updated PDI Header and Reset circuitry
Parts:
- added R?: 10k, ~, symbol R
- added SW?: RESET, ~, symbol SW_PUSH
Connections:
- wire segments 218 -> 223
- no-connect marks 5 -> 7
Other:
- note added: "Reset"
- moved on the sheet: P1
Changed lines of the file:
@@
 Text Label 8150 2700 0    60   ~ 0
 AIN0
-Text Notes 6500 1400 0    60   ~ 0
+Text Notes 6350 1400 0    60   ~ 0
 PDI Header
 $Comp
@@
 L CONN_3X2 P1
 U 1 1 4FA823D1
-P 7200 1700
-F 0 "P1" H 7200 1950 50  0000 C CNN
-F 1 "PDI" V 7200 1750 40  0000 C CNN
-F 2 "" H 7200 1700 60  0001 C CNN
-F 3 "" H 7200 1700 60  0001 C CNN
-	1    7200 1700
+P 7050 1700
+F 0 "P1" H 7050 1950 50  0000 C CNN
+F 1 "PDI" V 7050 1750 40  0000 C CNN
+F 2 "" H 7050 1700 60  0001 C CNN
+F 3 "" H 7050 1700 60  0001 C CNN
+	1    7050 1700
 	1    0    0    -1
 $EndComp
@@
 6E 56 52 49 51 4E 59 71 7E 65 C5 4D 0F AF 00 BF F6 21 9D BA 45 88 9C 00 16 00 C0 66 90 E0 00 00
 AC 42 3B 38 00 00 AB 90 E0 00 00 AC 42 82 03 00 B0 EA FF 00 E3 76 B5 A7 81 B6 BC 08 00 00 00 00
-49 45 4E 44 AE 42 60 82 E1 $EndBitmap
+49 45 4E 44 AE 42 60 82 C7 $EndBitmap
 EndData
 $EndBitmap
@@
 Text Notes 10900 2900 0    60   ~ 0
 Part should be specified\n(ZX62WRD-B-5PC). Water\nresistant USB Micro. Also,\nUSB Shield should be properly\nterminated.
-Text Notes 6550 1950 0    60   ~ 0
+Text Notes 6400 1950 0    60   ~ 0
 Update with PDI Header pins
 Text Notes 9000 6650 0    60   ~ 0
@@
 	10150 2250 10350 2250
 Wire Wire Line
-	7600 1650 7650 1650
-Wire Wire Line
-	6800 1550 6750 1550
-Wire Wire Line
-	6800 1750 6750 1750
+	7450 1650 7500 1650
+Wire Wire Line
+	6650 1550 6600 1550
+Wire Wire Line
+	6650 1750 6600 1750
 Wire Wire Line
 	14450 5550 14450 6450
@@
 	14450 6850 14450 8800
 Wire Wire Line
-	6800 1650 6750 1650
-Wire Wire Line
-	7600 1550 7650 1550
-Wire Wire Line
-	7600 1750 7650 1750
+	6650 1650 6600 1650
+Wire Wire Line
+	7450 1550 7500 1550
+Wire Wire Line
+	7450 1750 7500 1750
 Wire Notes Line
 	10750 1300 10750 3400
@@
 	11550 2500 11600 2500
 Wire Notes Line
-	6450 2000 7950 2000
+	6150 2000 7650 2000
 Wire Wire Line
 	9650 2250 9650 2200
@@
 	9750 2100 9750 2200
 Wire Notes Line
-	6450 1300 6450 2000
+	6150 1300 6150 2000
 Connection ~ 15150 2200
 $Comp
@@
 Text Label 850  3300 0    60   ~ 0
 XERR
+Text Label 6600 1550 2    60   ~ 0
+PDI_DATA
+Text Label 6600 1750 2    60   ~ 0
+PDI_CLK
+Text Label 7500 1550 0    60   ~ 0
+VCC
+$Comp
+L GND #PWR?
+U 1 1 5249BE44
+P 7500 1800
+F 0 "#PWR?" H 7500 1800 30  0001 C CNN
+F 1 "GND" H 7500 1730 30  0001 C CNN
+F 2 "" H 7500 1800 60  0000 C CNN
+F 3 "" H 7500 1800 60  0000 C CNN
+	1    7500 1800
+	1    0    0    -1
+$EndComp
+Wire Wire Line
+	7500 1750 7500 1800
+NoConn ~ 7500 1650
+NoConn ~ 6600 1650
+$Comp
+L R R?
+U 1 1 5249BF5B
+P 7300 2600
+F 0 "R?" V 7380 2600 40  0000 C CNN
+F 1 "10k" V 7307 2601 40  0000 C CNN
+F 2 "~" V 7230 2600 30  0000 C CNN
+F 3 "~" H 7300 2600 30  0000 C CNN
+	1    7300 2600
+	1    0    0    -1
+$EndComp
+$Comp
+L SW_PUSH SW?
+U 1 1 5249BF8D
+P 7300 3250
+F 0 "SW?" H 7450 3360 50  0000 C CNN
+F 1 "RESET" H 7300 3170 50  0000 C CNN
+F 2 "~" H 7300 3250 60  0000 C CNN
+F 3 "~" H 7300 3250 60  0000 C CNN
+	1    7300 3250
+	0    -1   -1   0
+$EndComp
+Wire Wire Line
+	7300 2850 7300 2950
+Wire Wire Line
+	7300 2350 7300 2300
+Text Label 7300 2300 2    60   ~ 0
+VCC
+Wire Wire Line
+	7300 2900 7250 2900
+Connection ~ 7300 2900
+Text Label 7250 2900 2    60   ~ 0
+PDI_CLK
+$Comp
+L GND #PWR?
+U 1 1 5249C2C6
+P 7300 3600
+F 0 "#PWR?" H 7300 3600 30  0001 C CNN
+F 1 "GND" H 7300 3530 30  0001 C CNN
+F 2 "" H 7300 3600 60  0000 C CNN
+F 3 "" H 7300 3600 60  0000 C CNN
+	1    7300 3600
+	1    0    0    -1
+$EndComp
+Wire Wire Line
+	7300 3550 7300 3600
+Text Notes 6950 2150 0    60   ~ 0
+Reset
 $EndSCHEMATC

Commit message: Added input power to uC, modified pins, added white LEDs and SPST switch, and made other small changes.
Parts:
- removed R4: 10k, symbol R
- removed S1: TL3315NF160Q, symbol TL3315NF160Q
- removed U2: USBMICRO-B, symbol USBMICRO-B
- added C?: 4.7nF, ~, symbol CSMALL
- added C? (x5): 0.1uF, ~, symbol CSMALL
- added C? (x2): 10uF, ~, symbol CSMALL
- added D? (x5): White LED, ~, symbol LED
- added J?: USB-MICRO-B, ~, symbol USB-MICRO-B
- added L? (x2): 10uH, ~, symbol INDUCTOR
- added R?: 1M, ~, symbol R
- added R? (x5): R, ~, symbol R
- added SW?: ON/OFF, ~, symbol SPSTSMALL
- gave numbers to parts that had none: 1
- renumbered C9 to C?, C12 to C?, C6 to C?, C7 to C?, C10 to C?, C8 to C?, C11 to C?, C13 to C?, C3 to C?, L2 to L?, P1 to P?, R5 to R?, S2 to S?, U3 to U?
Connections:
- net labels added: AS_MODE, MODE_SELECT, WL1, WL2, WL3, WL4, WL5
- net labels removed: MODE, SW?
- wire segments 223 -> 267
Other:
- note added: "AVR1017\nSection 3.3.3"
- note added: "Ferrite Bead\nAVR1012\nSection 2.1"
- note added: "White LEDs\n(Placed between\nRGB LEDs)"
- note added: "ZX62WRD-B-5PC"
- note removed: "Part should be specified\n(ZX62WRD-B-5PC). Water\nresistant USB Micro. Also,\nUSB Shield should be properly\nterminated."
- moved on the sheet: BT1, D7, F?, L?, R?, S?, TP1, TP2, U?

Commit message: Finalized (for now) the schematics and annotated components.
Parts:
- added R11, R13, R15, R16, R17, R18, R2, R20, R21, R4, R9: 10k, ~, symbol R
- BEAD1: renamed from L?; value 10uH -> Ferrite
- R10, R12, R14, R3, R5: renamed from R?; value R -> 120
- gave numbers to parts that had none: 44
Connections:
- net labels added: PD0, PD1, PD10, PD2, PD3, PD4, PD5, PD6, PD7, PD8, PD9
- wire segments 267 -> 300
Other:
- note added: "Pull-Down Resistors"
- note removed: "Import smaller RGB LED\nfrom Pong.0"
- note removed: "Update with PDI Header pins"
- moved on the sheet: BEAD1, D10, D11, D12, D8, D9, L1, P1, R1, R10, R12, R14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

Commit message: Added latching power block
Parts:
- removed SW2: ON/OFF, ~, symbol SPSTSMALL
- removed TP2: TST, symbol TST
- added C20: 1uF, ~, symbol CSMALL
- added C21: 0.1uF, ~, symbol CSMALL
- added C22: 10uF, ~, symbol CSMALL
- added D13: DIODE, ~, symbol DIODE
- added R25: 10k, ~, symbol R
- added R26, R28: 100k, ~, symbol R
- added R27: 300k, ~, symbol R
- added SW2: ON_OFF, ~, symbol SW_PUSH
- added U5: SI3588DV, symbol SI3588DV
Connections:
- wire segments 300 -> 319
Other:
- note added: "Latching Power Block\nFrom Mosaic Industries\nApp Notes"
- moved on the sheet: BEAD1, BT1, D10, D11, D12, D7, D8, D9, F1, J1, L1, L2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
